Commit message: feat(variobot_description): Add 48mm_N20_Mecanum_Drive_Base

File: variobot_description/description/sdf/model.sdf.xacro (robot description, xacro)
@@ -5,10 +5,6 @@
       <must_be_base_link>true</must_be_base_link>
     </link>
-    <joint name="base_footprint_joint" type="fixed">
-      <pose relative_to="base_link"/>
-      <parent>base_link</parent>
-      <child>base_footprint_link</child>
-    </joint>
-    <link name="base_footprint_link"/>
+    <xacro:include
+      filename="mobility_systems/mecanum_drive/48mm_n20_mecanum_drive/48mm_n20_mecanum_drive.sdf.xacro" />
   </model>
 </sdf>

Commit message: feat(variobot_description): Add 48mm_N20_Mecanum_Drive Mobility System (#12)

File: variobot_description/description/sdf/model.sdf.xacro (robot description, xacro)
@@ -1,14 +1,10 @@
 <?xml version="1.0"?>
-<sdf version="1.11" xmlns:xacro="http://www.ros.org/wiki/xacro">
+<sdf version="1.12" xmlns:xacro="http://www.ros.org/wiki/xacro">
   <model name="variobot" canonical_link="base_link">
     <link name="base_link">
       <must_be_base_link>true</must_be_base_link>
     </link>
-    <joint name="base_footprint_joint" type="fixed">
-      <pose relative_to="base_link"/>
-      <parent>base_link</parent>
-      <child>base_footprint_link</child>
-    </joint>
-    <link name="base_footprint_link"/>
+    <xacro:include
+      filename="mobility_systems/mecanum_drive/48mm_n20_mecanum_drive/48mm_n20_mecanum_drive.sdf.xacro" />
   </model>
 </sdf>
