Commit message: Complete 48mm_N20_Mecanum_Drive robot description

File: variobot_description/description/sdf/mobility_systems/mecanum_drive/48mm_n20_mecanum_drive/48mm_n20_mecanum_drive.sdf.xacro (robot description, xacro)
@@ -9,4 +9,5 @@
     <pose relative_to="mobility_system_joint" />
     <visual name="mobility_system_visual">
+      <pose relative_to="mobility_system_link" degrees="true">0 0 0 0 0 -90</pose>
       <geometry>
         <mesh>
@@ -28,3 +29,367 @@
     <inertial auto="true" />
   </link>
+  <joint name="front_left_motor_joint" type="fixed">
+    <pose relative_to="mobility_system_link" degrees="true">0.05 0.0759 0.009 0 0 -90</pose>
+    <parent>mobility_system_link</parent>
+    <child>front_left_motor_link</child>
+  </joint>
+  <link name="front_left_motor_link">
+    <pose relative_to="front_left_motor_joint" />
+    <visual name="front_left_motor_visual">
+      <pose relative_to="front_left_motor_link" />
+      <geometry>
+        <mesh>
+          <uri>
+            package://variobot_description/meshes/Motors/N20_Motor/N20_Motor_Assembly_Left.dae
+          </uri>
+        </mesh>
+      </geometry>
+    </visual>
+    <collision name="front_left_motor_collision">
+      <pose relative_to="front_left_motor_link" />
+      <geometry>
+        <box>
+          <size>0.024 0.0248 0.012</size>
+        </box>
+      </geometry>
+    </collision>
+    <inertial auto="true" />
+  </link>
+  <joint name="front_left_coupling_joint" type="revolute">
+    <pose relative_to="front_left_motor_link" degrees="true">0.02305 0 -0.001 0 0 0</pose>
+    <parent>front_left_motor_link</parent>
+    <child>front_left_coupling_link</child>
+    <axis>
+      <xyz>1 0 0</xyz>
+      <limit>
+        <lower>-inf</lower>
+        <upper>inf</upper>
+        <velocity>31.41</velocity>
+      </limit>
+    </axis>
+  </joint>
+  <link name="front_left_coupling_link">
+    <pose relative_to="front_left_coupling_joint" />
+    <visual name="front_left_coupling_visual">
+      <pose relative_to="front_left_coupling_link" degrees="true">0 0 0 0 0 90</pose>
+      <geometry>
+        <mesh>
+          <uri>
+            package://variobot_description/meshes/Mobility_Systems/Mecanum_Drive/48mm_N20_Mecanum_Drive/48mm_Mecanum_Wheel_N20_Motor_Coupling.dae
+          </uri>
+        </mesh>
+      </geometry>
+    </visual>
+    <collision name="front_left_coupling_collision">
+      <pose relative_to="front_left_coupling_link" degrees="true">-0.004 0 0 0 90 0</pose>
+      <geometry>
+        <cylinder>
+          <radius>0.00507</radius>
+          <length>0.012</length>
+        </cylinder>
+      </geometry>
+    </collision>
+    <inertial auto="true" />
+  </link>
+  <joint name="front_left_wheel_joint" type="fixed">
+    <pose relative_to="front_left_coupling_link">0.01915 0 0 0 0 0</pose>
+    <parent>front_left_coupling_link</parent>
+    <child>front_left_wheel_link</child>
+  </joint>
+  <link name="front_left_wheel_link">
+    <pose relative_to="front_left_wheel_joint" />
+    <visual name="front_left_wheel_visual">
+      <pose relative_to="front_left_wheel_link" degrees="true">0 0 0 0 0 -90</pose>
+      <geometry>
+        <mesh>
+          <uri>
+            package://variobot_description/meshes/Mobility_Systems/Mecanum_Drive/48mm_N20_Mecanum_Drive/48mm_Mecanum_Wheel_Left.dae
+          </uri>
+        </mesh>
+      </geometry>
+    </visual>
+    <collision name="front_left_wheel_collision">
+      <pose relative_to="front_left_coupling_link" degrees="true">0.01285 0 0 0 90 0</pose>
+      <geometry>
+        <cylinder>
+          <radius>0.024</radius>
+          <length>0.025</length>
+        </cylinder>
+      </geometry>
+    </collision>
+    <inertial auto="true" />
+  </link>
+  <joint name="front_right_motor_joint" type="fixed">
+    <pose relative_to="mobility_system_link" degrees="true">0.05 -0.0759 0.009 0 0 90</pose>
+    <parent>mobility_system_link</parent>
+    <child>front_right_motor_link</child>
+  </joint>
+  <link name="front_right_motor_link">
+    <pose relative_to="front_right_motor_joint" />
+    <visual name="front_right_motor_visual">
+      <pose relative_to="front_right_motor_link" degrees="true">0 0 0 0 0 180</pose>
+      <geometry>
+        <mesh>
+          <uri>
+            package://variobot_description/meshes/Motors/N20_Motor/N20_Motor_Assembly_Right.dae
+          </uri>
+        </mesh>
+      </geometry>
+    </visual>
+    <collision name="front_right_motor_collision">
+      <pose relative_to="front_right_motor_link" />
+      <geometry>
+        <box>
+          <size>0.024 0.0248 0.012</size>
+        </box>
+      </geometry>
+    </collision>
+    <inertial auto="true" />
+  </link>
+  <joint name="front_right_coupling_joint" type="revolute">
+    <pose relative_to="front_right_motor_link" degrees="true">0.02305 0 -0.001 0 0 0</pose>
+    <parent>front_right_motor_link</parent>
+    <child>front_right_coupling_link</child>
+    <axis>
+      <xyz>1 0 0</xyz>
+      <limit>
+        <lower>-inf</lower>
+        <upper>inf</upper>
+        <velocity>31.41</velocity>
+      </limit>
+    </axis>
+  </joint>
+  <link name="front_right_coupling_link">
+    <pose relative_to="front_right_coupling_joint" />
+    <visual name="front_right_coupling_visual">
+      <pose relative_to="front_right_coupling_link" degrees="true">0 0 0 0 0 90</pose>
+      <geometry>
+        <mesh>
+          <uri>
+            package://variobot_description/meshes/Mobility_Systems/Mecanum_Drive/48mm_N20_Mecanum_Drive/48mm_Mecanum_Wheel_N20_Motor_Coupling.dae
+          </uri>
+        </mesh>
+      </geometry>
+    </visual>
+    <collision name="front_right_coupling_collision">
+      <pose relative_to="front_right_coupling_link" degrees="true">-0.004 0 0 0 90 0</pose>
+      <geometry>
+        <cylinder>
+          <radius>0.00507</radius>
+          <length>0.012</length>
+        </cylinder>
+      </geometry>
+    </collision>
+    <inertial auto="true" />
+  </link>
+  <joint name="front_right_wheel_joint" type="fixed">
+    <pose relative_to="front_right_coupling_link">0.01915 0 0 0 0 0</pose>
+    <parent>front_right_coupling_link</parent>
+    <child>front_right_wheel_link</child>
+  </joint>
+  <link name="front_right_wheel_link">
+    <pose relative_to="front_right_wheel_joint" />
+    <visual name="front_right_wheel_visual">
+      <pose relative_to="front_right_wheel_link" degrees="true">0 0 0 0 0 -90</pose>
+      <geometry>
+        <mesh>
+          <uri>
+            package://variobot_description/meshes/Mobility_Systems/Mecanum_Drive/48mm_N20_Mecanum_Drive/48mm_Mecanum_Wheel_Right.dae
+          </uri>
+        </mesh>
+      </geometry>
+    </visual>
+    <collision name="front_right_wheel_collision">
+      <pose relative_to="front_right_coupling_link" degrees="true">0.01285 0 0 0 90 0</pose>
+      <geometry>
+        <cylinder>
+          <radius>0.024</radius>
+          <length>0.025</length>
+        </cylinder>
+      </geometry>
+    </collision>
+    <inertial auto="true" />
+  </link>
+  <joint name="rear_left_motor_joint" type="fixed">
+    <pose relative_to="mobility_system_link" degrees="true">-0.05 0.0759 0.009 0 0 -90</pose>
+    <parent>mobility_system_link</parent>
+    <child>rear_left_motor_link</child>
+  </joint>
+  <link name="rear_left_motor_link">
+    <pose relative_to="rear_left_motor_joint" />
+    <visual name="rear_left_motor_visual">
+      <pose relative_to="rear_left_motor_link" degrees="true">0 0 0 0 0 180</pose>
+      <geometry>
+        <mesh>
+          <uri>
+            package://variobot_description/meshes/Motors/N20_Motor/N20_Motor_Assembly_Right.dae
+          </uri>
+        </mesh>
+      </geometry>
+    </visual>
+    <collision name="rear_left_motor_collision">
+      <pose relative_to="rear_left_motor_link" />
+      <geometry>
+        <box>
+          <size>0.024 0.0248 0.012</size>
+        </box>
+      </geometry>
+    </collision>
+    <inertial auto="true" />
+  </link>
+  <joint name="rear_left_coupling_joint" type="revolute">
+    <pose relative_to="rear_left_motor_link" degrees="true">0.02305 0 -0.001 0 0 0</pose>
+    <parent>rear_left_motor_link</parent>
+    <child>rear_left_coupling_link</child>
+    <axis>
+      <xyz>1 0 0</xyz>
+      <limit>
+        <lower>-inf</lower>
+        <upper>inf</upper>
+        <velocity>31.41</velocity>
+      </limit>
+    </axis>
+  </joint>
+  <link name="rear_left_coupling_link">
+    <pose relative_to="rear_left_coupling_joint" />
+    <visual name="rear_left_coupling_visual">
+      <pose relative_to="rear_left_coupling_link" degrees="true">0 0 0 0 0 90</pose>
+      <geometry>
+        <mesh>
+          <uri>
+            package://variobot_description/meshes/Mobility_Systems/Mecanum_Drive/48mm_N20_Mecanum_Drive/48mm_Mecanum_Wheel_N20_Motor_Coupling.dae
+          </uri>
+        </mesh>
+      </geometry>
+    </visual>
+    <collision name="rear_left_coupling_collision">
+      <pose relative_to="rear_left_coupling_link" degrees="true">-0.004 0 0 0 90 0</pose>
+      <geometry>
+        <cylinder>
+          <radius>0.00507</radius>
+          <length>0.012</length>
+        </cylinder>
+      </geometry>
+    </collision>
+    <inertial auto="true" />
+  </link>
+  <joint name="rear_left_wheel_joint" type="fixed">
+    <pose relative_to="rear_left_coupling_link">0.01915 0 0 0 0 0</pose>
+    <parent>rear_left_coupling_link</parent>
+    <child>rear_left_wheel_link</child>
+  </joint>
+  <link name="rear_left_wheel_link">
+    <pose relative_to="rear_left_wheel_joint" />
+    <visual name="rear_left_wheel_visual">
+      <pose relative_to="rear_left_wheel_link" degrees="true">0 0 0 0 0 -90</pose>
+      <geometry>
+        <mesh>
+          <uri>
+            package://variobot_description/meshes/Mobility_Systems/Mecanum_Drive/48mm_N20_Mecanum_Drive/48mm_Mecanum_Wheel_Left.dae
+          </uri>
+        </mesh>
+      </geometry>
+    </visual>
+    <collision name="rear_left_wheel_collision">
+      <pose relative_to="rear_left_coupling_link" degrees="true">0.01285 0 0 0 90 0</pose>
+      <geometry>
+        <cylinder>
+          <radius>0.024</radius>
+          <length>0.025</length>
+        </cylinder>
+      </geometry>
+    </collision>
+    <inertial auto="true" />
+  </link>
+  <joint name="rear_right_motor_joint" type="fixed">
+    <pose relative_to="mobility_system_link" degrees="true">-0.05 -0.0759 0.009 0 0 90</pose>
+    <parent>mobility_system_link</parent>
+    <child>rear_right_motor_link</child>
+  </joint>
+  <link name="rear_right_motor_link">
+    <pose relative_to="rear_right_motor_joint" />
+    <visual name="rear_right_motor_visual">
+      <pose relative_to="rear_right_motor_link" />
+      <geometry>
+        <mesh>
+          <uri>
+            package://variobot_description/meshes/Motors/N20_Motor/N20_Motor_Assembly_Left.dae
+          </uri>
+        </mesh>
+      </geometry>
+    </visual>
+    <collision name="rear_right_motor_collision">
+      <pose relative_to="rear_right_motor_link" />
+      <geometry>
+        <box>
+          <size>0.024 0.0248 0.012</size>
+        </box>
+      </geometry>
+    </collision>
+    <inertial auto="true" />
+  </link>
+  <joint name="rear_right_coupling_joint" type="revolute">
+    <pose relative_to="rear_right_motor_link" degrees="true">0.02305 0 -0.001 0 0 0</pose>
+    <parent>rear_right_motor_link</parent>
+    <child>rear_right_coupling_link</child>
+    <axis>
+      <xyz>1 0 0</xyz>
+      <limit>
+        <lower>-inf</lower>
+        <upper>inf</upper>
+        <velocity>31.41</velocity>
+      </limit>
+    </axis>
+  </joint>
+  <link name="rear_right_coupling_link">
+    <pose relative_to="rear_right_coupling_joint" />
+    <visual name="rear_right_coupling_visual">
+      <pose relative_to="rear_right_coupling_link" degrees="true">0 0 0 0 0 90</pose>
+      <geometry>
+        <mesh>
+          <uri>
+            package://variobot_description/meshes/Mobility_Systems/Mecanum_Drive/48mm_N20_Mecanum_Drive/48mm_Mecanum_Wheel_N20_Motor_Coupling.dae
+          </uri>
+        </mesh>
+      </geometry>
+    </visual>
+    <collision name="rear_right_coupling_collision">
+      <pose relative_to="rear_right_coupling_link" degrees="true">-0.004 0 0 0 90 0</pose>
+      <geometry>
+        <cylinder>
+          <radius>0.00507</radius>
+          <length>0.012</length>
+        </cylinder>
+      </geometry>
+    </collision>
+    <inertial auto="true" />
+  </link>
+  <joint name="rear_right_wheel_joint" type="fixed">
+    <pose relative_to="rear_right_coupling_link">0.01915 0 0 0 0 0</pose>
+    <parent>rear_right_coupling_link</parent>
+    <child>rear_right_wheel_link</child>
+  </joint>
+  <link name="rear_right_wheel_link">
+    <pose relative_to="rear_right_wheel_joint" />
+    <visual name="rear_right_wheel_visual">
+      <pose relative_to="rear_right_wheel_link" degrees="true">0 0 0 0 0 -90</pose>
+      <geometry>
+        <mesh>
+          <uri>
+            package://variobot_description/meshes/Mobility_Systems/Mecanum_Drive/48mm_N20_Mecanum_Drive/48mm_Mecanum_Wheel_Right.dae
+          </uri>
+        </mesh>
+      </geometry>
+    </visual>
+    <collision name="rear_right_wheel_collision">
+      <pose relative_to="rear_right_coupling_link" degrees="true">0.01285 0 0 0 90 0</pose>
+      <geometry>
+        <cylinder>
+          <radius>0.024</radius>
+          <length>0.025</length>
+        </cylinder>
+      </geometry>
+    </collision>
+    <inertial auto="true" />
+  </link>
 </sdf>

Commit message: feat(variobot_control and variobot_gz): Add 48mm_N20_Mecanum_Drive Mobility System

File: variobot_description/description/sdf/mobility_systems/mecanum_drive/48mm_n20_mecanum_drive/48mm_n20_mecanum_drive.sdf.xacro (robot description, xacro)
@@ -1,4 +1,5 @@
 <?xml version="1.0"?>
-<sdf version="1.12" xmlns:xacro="http://www.ros.org/wiki/xacro">
+<sdf version="1.12" xmlns:xacro="http://www.ros.org/wiki/xacro"
+  xmlns:gz="http://gazebosim.org/schema">
   <joint name="mobility_system_joint" type="fixed">
     <pose relative_to="base_link" />
@@ -61,5 +62,5 @@
     <child>front_left_coupling_link</child>
     <axis>
-      <xyz>1 0 0</xyz>
+      <xyz>-1 0 0</xyz>
       <limit>
         <lower>-inf</lower>
@@ -117,4 +118,13 @@
         </cylinder>
       </geometry>
+      <surface>
+        <friction>
+          <ode>
+            <mu>1.0</mu>
+            <mu2>0.0</mu2>
+            <fdir1 gz:expressed_in="base_link">1 -1 0</fdir1>
+          </ode>
+        </friction>
+      </surface>
     </collision>
     <inertial auto="true" />
@@ -208,4 +218,13 @@
         </cylinder>
       </geometry>
+      <surface>
+        <friction>
+          <ode>
+            <mu>1.0</mu>
+            <mu2>0.0</mu2>
+            <fdir1 gz:expressed_in="base_link">1 1 0</fdir1>
+          </ode>
+        </friction>
+      </surface>
     </collision>
     <inertial auto="true" />
@@ -243,5 +262,5 @@
     <child>rear_left_coupling_link</child>
     <axis>
-      <xyz>1 0 0</xyz>
+      <xyz>-1 0 0</xyz>
       <limit>
         <lower>-inf</lower>
@@ -299,4 +318,13 @@
         </cylinder>
       </geometry>
+      <surface>
+        <friction>
+          <ode>
+            <mu>1.0</mu>
+            <mu2>0.0</mu2>
+            <fdir1 gz:expressed_in="base_link">1 1 0</fdir1>
+          </ode>
+        </friction>
+      </surface>
     </collision>
     <inertial auto="true" />
@@ -390,6 +418,17 @@
         </cylinder>
       </geometry>
-    </collision>
-    <inertial auto="true" />
-  </link>
+      <surface>
+        <friction>
+          <ode>
+            <mu>1.0</mu>
+            <mu2>0.0</mu2>
+            <fdir1 gz:expressed_in="base_link">1 -1 0</fdir1>
+          </ode>
+        </friction>
+      </surface>
+    </collision>
+    <inertial auto="true" />
+  </link>
+  <xacro:include
+    filename="$(find variobot_control)/description/sdf/mobility_systems/mecanum_drive/48mm_n20_mecanum_drive/gz_ros2_control.sdf.xacro" />
 </sdf>

Commit message: feat(gz): Make RPLidar work in simulation

File: variobot_description/description/sdf/mobility_systems/mecanum_drive/48mm_n20_mecanum_drive/48mm_n20_mecanum_drive.sdf.xacro (robot description, xacro)
@@ -430,4 +430,10 @@
     <inertial auto="true" />
   </link>
+  <joint name="lidar_base_joint" type="fixed">
+    <pose relative_to="mobility_system_link" degrees="true">0 0 0.035 0 0 0</pose>
+    <parent>mobility_system_link</parent>
+    <child>lidar_base_link</child>
+  </joint>
+  <xacro:include filename="$(find variobot_description)/description/sdf/lidar_parts/lidar.sdf.xacro" />
   <xacro:include
     filename="$(find variobot_control)/description/sdf/mobility_systems/mecanum_drive/48mm_n20_mecanum_drive/ros2_control.sdf.xacro" />

File: variobot_gz/worlds/common_elements.sdf.xacro (robot description, xacro)
@@ -1,4 +1,5 @@
 <?xml version="1.0"?>
 <sdf version="1.12">
+  <plugin filename="gz-sim-sensors-system" name="gz::sim::systems::Sensors" />
   <plugin filename="gz-sim-user-commands-system" name="gz::sim::systems::UserCommands" />
   <physics type="dart" />

Commit message: feat(sensors): Add RPLidar A1 M8 (#22)

File: variobot_description/description/sdf/mobility_systems/mecanum_drive/48mm_n20_mecanum_drive/48mm_n20_mecanum_drive.sdf.xacro (robot description, xacro)
@@ -430,4 +430,10 @@
     <inertial auto="true" />
   </link>
+  <joint name="lidar_base_joint" type="fixed">
+    <pose relative_to="mobility_system_link" degrees="true">0 0 0.035 0 0 0</pose>
+    <parent>mobility_system_link</parent>
+    <child>lidar_base_link</child>
+  </joint>
+  <xacro:include filename="$(find variobot_description)/description/sdf/lidar_parts/lidar.sdf.xacro" />
   <xacro:include
     filename="$(find variobot_control)/description/sdf/mobility_systems/mecanum_drive/48mm_n20_mecanum_drive/ros2_control.sdf.xacro" />
